Commit message: finished setting up the diff drive plugin

File: rb1_ros2_description/xacro/rb1_ros2_base.urdf.xacro (robot description, xacro)
@@ -85,4 +85,36 @@
 	</xacro:sensor_orbbec_astra>
 	<!-- Gazebo ros2 control plugins -->
+    <ros2_control name="GazeboSystem" type="system">
+        <hardware>
+            <plugin>gazebo_ros2_control/GazeboSystem</plugin>
+        </hardware>
+        <joint name="$(arg prefix)right_wheel_joint">
+            <command_interface name="velocity">
+                <param name="min">-1</param>
+                <param name="max">1</param>
+            </command_interface>
+            <state_interface name="position"/>
+            <state_interface name="velocity"/>
+            <state_interface name="effort"/>
+        </joint>
+        <joint name="$(arg prefix)left_wheel_joint">
+            <command_interface name="velocity">
+                <param name="min">-1</param>
+                <param name="max">1</param>
+            </command_interface>
+            <state_interface name="position"/>
+            <state_interface name="velocity"/>
+            <state_interface name="effort"/>
+        </joint>
+    </ros2_control>
+    <gazebo>
+        <plugin filename="libgazebo_ros2_control.so" name="gazebo_ros2_control">
+            <ros>
+                <namespace>rb1_robot</namespace>
+            </ros>
+            <robot_sim_type>gazebo_ros2_control/GazeboSystem</robot_sim_type>
+            <parameters>$(find rb1_ros2_description)/config/rb1_controller.yaml</parameters>
+        </plugin>
+    </gazebo>
 	<!-- <xacro:ros2_control/> -->
 </robot>

Commit message: finished elevator joint

File: rb1_ros2_description/xacro/rb1_ros2_base.urdf.xacro (robot description, xacro)
@@ -107,4 +107,13 @@
             <state_interface name="effort"/>
         </joint>
+        <!-- <joint name="robot_elevator_base_joint">
+            <command_interface name="position">
+                <param name="min">-1</param>
+                <param name="max">1</param>
+            </command_interface>
+            <state_interface name="position"/>
+            <state_interface name="velocity"/>
+            <state_interface name="effort"/>
+        </joint> -->
     </ros2_control>
     <gazebo>
@@ -117,4 +126,15 @@
         </plugin>
     </gazebo>
+    <gazebo>
+        <plugin name="gazebo_ros_force" filename="libgazebo_ros_force.so">
+            <!-- <ros>
+                <namespace>rb1_robot</namespace>
+            </ros> -->
+             <!-- Name of link within model which will receive the force -->
+            <link_name>robot_elevator_platform_link</link_name>
+            <!-- Frame where the force/torque will be applied (options: world; link)-->
+            <force_frame>link</force_frame>
+        </plugin>
+    </gazebo>
 	<!-- <xacro:ros2_control/> -->
 </robot>
